Commit message: Update sensor.urdf.xacro

File: pr2_robot/urdf/sensor.urdf.xacro (robot description, xacro)
@@ -12,5 +12,5 @@
     <origin xyz="0 0 0" rpy="0 0 0"/>
     <geometry>
-      <mesh filename="package://sensor_stick/meshes/asus_xtion.dae"/>
+      <mesh filename="package://pr2_robot/models/asus_xtion.dae"/>
     </geometry>
   </visual>
